Commit message: latest stable

File: config/robot.urdf.xacro (robot description, xacro)
@@ -2,32 +2,38 @@
 <robot name="lio" xmlns:xacro="http://tixiaoshan.github.io/">
   <xacro:property name="PI" value="3.1415926535897931" />
-  <link name="chassis_link"></link>
+  <link name="world"></link>
+  <link name="odom"></link>
+  <joint name="odom_joint" type="fixed">
+    <parent link="world" />
+    <child link="odom" />
+    <origin xyz="0 0 0" rpy="0 0 0" />
+  </joint>
   <link name="base_link"></link>
   <joint name="base_link_joint" type="fixed">
-    <parent link="base_link"/>
-    <child link="chassis_link" />
+    <parent link="world" />
+    <child link="base_link" />
     <origin xyz="0 0 0" rpy="0 0 0" />
   </joint>
-  <link name="lidar_link"> </link>
+  <link name="velodyne"> </link>
   <joint name="lidar_joint" type="fixed">
     <parent link="base_link" />
-    <child link="lidar_link" />
-    <origin xyz="0 0 0" rpy="0 0 0" />
+    <child link="velodyne" />
+    <origin xyz="0 0 -0.21" rpy="0 0 0" />
   </joint>
   <link name="imu_link"> </link>
   <joint name="imu_joint" type="fixed">
-    <parent link="chassis_link" />
+    <parent link="velodyne" />
     <child link="imu_link" />
-    <origin xyz="0 0 0" rpy="0 0 0" />
+    <origin xyz="0.003 0.25536 -0.21" rpy="0 0 -90" />
   </joint>
-  <link name="laser_sensor_frame"> </link>
-  <joint name="laser_joint" type="fixed">
-    <parent link="imu_link" />
-    <child link="laser_sensor_frame" />
-    <origin xyz="0 0 0" rpy="0 0 0" />
+  <link name="map-centric"> </link>
+  <joint name="map_joint_joint" type="fixed">
+    <parent link="base_link" />
+    <child link="map-centric" />
+    <origin xyz="0 0 -0.21" rpy="0 0 0" />
   </joint>
   <link name="navsat_link"> </link>
   <joint name="navsat_joint" type="fixed">
-    <parent link="chassis_link" />
+    <parent link="odom" />
     <child link="navsat_link" />
     <origin xyz="0 0 0" rpy="0 0 0" />

Commit message: 01/06/2024

File: config/robot.urdf.xacro (robot description, xacro)
@@ -21,8 +21,8 @@
     <origin xyz="0 0 -0.21" rpy="0 0 0" />
   </joint>
-  <link name="imu_link"> </link>
+  <link name="imu_link1"> </link>
   <joint name="imu_joint" type="fixed">
     <parent link="velodyne" />
-    <child link="imu_link" />
+    <child link="imu_link1" />
     <origin xyz="0.003 0.25536 -0.21" rpy="0 0 -90" />
   </joint>

Commit message: 15/06/2024

File: config/robot.urdf.xacro (robot description, xacro)
@@ -2,8 +2,8 @@
 <robot name="lio" xmlns:xacro="http://tixiaoshan.github.io/">
   <xacro:property name="PI" value="3.1415926535897931" />
-  <link name="world"></link>
+  <link name="map"></link>
   <link name="odom"></link>
   <joint name="odom_joint" type="fixed">
-    <parent link="world" />
+    <parent link="map" />
     <child link="odom" />
     <origin xyz="0 0 0" rpy="0 0 0" />

Commit message: 23/06/2024

File: config/robot.urdf.xacro (robot description, xacro)
@@ -11,5 +11,5 @@
   <link name="base_link"></link>
   <joint name="base_link_joint" type="fixed">
-    <parent link="world" />
+    <parent link="map" />
     <child link="base_link" />
     <origin xyz="0 0 0" rpy="0 0 0" />

Commit message: 29/06/2024

File: config/robot.urdf.xacro (robot description, xacro)
@@ -1,41 +1,171 @@
-<?xml version="1.0"?>
-<robot name="lio" xmlns:xacro="http://tixiaoshan.github.io/">
-  <xacro:property name="PI" value="3.1415926535897931" />
-  <link name="map"></link>
-  <link name="odom"></link>
-  <joint name="odom_joint" type="fixed">
-    <parent link="map" />
-    <child link="odom" />
+<robot name="scout_v2">
+  <!-- Base link -->
+  <link name="base_link">
+    <visual>
+      <origin rpy="0 0 0" xyz="0 0 0"/>
+      <geometry>
+        <mesh filename="package://scout_description/meshes/scout_v2/base_link.dae"/>
+      </geometry>
+    </visual>
+    <collision>
+      <origin rpy="0 0 0" xyz="0 0 0.008"/>
+      <geometry>
+        <box size="0.925 0.38 0.21"/>
+      </geometry>
+    </collision>
+    <collision>
+      <origin rpy="0 0 0" xyz="0 0 0.034999999999999996"/>
+      <geometry>
+        <box size="0.15416666666666667 0.627 0.06999999999999999"/>
+      </geometry>
+    </collision>
+  </link>
+  <link name="Rs_lidar"> </link>
+  <joint name="lidar_joint" type="fixed">
+    <parent link="base_link" />
+    <child link="Rs_lidar" />
+    <origin xyz="0 0 0.23" rpy="0 0 0" />
+  </joint>
+  <link name="rslidar"> </link>
+  <joint name="rslidar_joint" type="fixed">
+    <parent link="Rs_lidar" />
+    <child link="rslidar" />
     <origin xyz="0 0 0" rpy="0 0 0" />
   </joint>
-  <link name="base_link"></link>
-  <joint name="base_link_joint" type="fixed">
-    <parent link="map" />
-    <child link="base_link" />
-    <origin xyz="0 0 0" rpy="0 0 0" />
-  </joint>
-  <link name="velodyne"> </link>
-  <joint name="lidar_joint" type="fixed">
+  <link name="map_centric"> </link>
+  <joint name="map_centric_joint" type="fixed">
     <parent link="base_link" />
-    <child link="velodyne" />
-    <origin xyz="0 0 -0.21" rpy="0 0 0" />
+    <child link="map_centric" />
+    <origin xyz="0 0 -0.432051" rpy="0 0 0" />
   </joint>
   <link name="imu_link"> </link>
   <joint name="imu_joint" type="fixed">
-    <parent link="velodyne" />
+    <parent link="base_link" />
     <child link="imu_link" />
-    <origin xyz="0.003 0.25536 -0.21" rpy="0 0 -90" />
-  </joint>
-  <link name="map-centric"> </link>
-  <joint name="map_joint_joint" type="fixed">
-    <parent link="base_link" />
-    <child link="map-centric" />
-    <origin xyz="0 0 -0.21" rpy="0 0 0" />
+    <origin xyz="0.25536 0.003 0.02" rpy="0 0 0" />
   </joint>
   <link name="navsat_link"> </link>
   <joint name="navsat_joint" type="fixed">
-    <parent link="odom" />
+    <parent link="base_link" />
     <child link="navsat_link" />
-    <origin xyz="0 0 0" rpy="0 0 0" />
+    <origin xyz="0.003 0.25536 0.07" rpy="0 0 0" />
+  </joint>
+  <link name="base_footprint"/>
+  <joint name="base_footprint_joint" type="fixed">
+    <origin rpy="0 0 0" xyz="0 0 -0.23479"/>
+    <parent link="base_link"/>
+    <child link="base_footprint"/>
+  </joint>
+  <link name="inertial_link">
+    <inertial>
+      <mass value="40"/>
+      <origin xyz="0.0 0.0 0.0"/>
+      <inertia ixx="2.288641" ixy="0" ixz="0" iyy="5.103976" iyz="0" izz="3.431465"/>
+    </inertial>
+  </link>
+  <joint name="inertial_joint" type="fixed">
+    <origin rpy="0 0 0" xyz="0 0 0"/>
+    <parent link="base_link"/>
+    <child link="inertial_link"/>
+  </joint>
+  <link name="front_right_wheel_link">
+    <inertial>
+      <mass value="3"/>
+      <origin xyz="0 0 0"/>
+      <inertia ixx="0.7171" ixy="0" ixz="0" iyy="0.1361" iyz="0" izz="0.7171"/>
+    </inertial>
+    <visual>
+      <origin rpy="0 0 0" xyz="0 0 0"/>
+      <geometry>
+        <mesh filename="package://scout_description/meshes/scout_v2/wheel_type1.dae"/>
+      </geometry>
+    </visual>
+    <collision>
+      <origin rpy="1.570795 0 0" xyz="0 0 0"/>
+      <geometry>
+        <cylinder length="0.11653" radius="0.16459"/>
+      </geometry>
+    </collision>
+  </link>
+  <joint name="front_right_wheel" type="fixed">
+    <parent link="base_link"/>
+    <child link="front_right_wheel_link"/>
+    <origin rpy="3.14 0 0" xyz="0.249 -0.29153 -0.0702"/>
+    <axis rpy="0 0 0" xyz="0 -1 0"/>
+  </joint>
+  <link name="front_left_wheel_link">
+    <inertial>
+      <mass value="3"/>
+      <origin xyz="0 0 0"/>
+      <inertia ixx="0.7171" ixy="0" ixz="0" iyy="0.1361" iyz="0" izz="0.7171"/>
+    </inertial>
+    <visual>
+      <origin rpy="0 0 0" xyz="0 0 0"/>
+      <geometry>
+        <mesh filename="package://scout_description/meshes/scout_v2/wheel_type2.dae"/>
+      </geometry>
+    </visual>
+    <collision>
+      <origin rpy="1.570795 0 0" xyz="0 0 0"/>
+      <geometry>
+        <cylinder length="0.11653" radius="0.16459"/>
+      </geometry>
+    </collision>
+  </link>
+  <joint name="front_left_wheel" type="fixed">
+    <parent link="base_link"/>
+    <child link="front_left_wheel_link"/>
+    <origin rpy="0 0 0" xyz="0.249 0.29153 -0.0702"/>
+    <axis rpy="0 0 0" xyz="0 -1 0"/>
+  </joint>
+  <link name="rear_left_wheel_link">
+    <inertial>
+      <mass value="3"/>
+      <origin xyz="0 0 0"/>
+      <inertia ixx="0.7171" ixy="0" ixz="0" iyy="0.1361" iyz="0" izz="0.7171"/>
+    </inertial>
+    <visual>
+      <origin rpy="0 0 0" xyz="0 0 0"/>
+      <geometry>
+        <mesh filename="package://scout_description/meshes/scout_v2/wheel_type1.dae"/>
+      </geometry>
+    </visual>
+    <collision>
+      <origin rpy="1.570795 0 0" xyz="0 0 0"/>
+      <geometry>
+        <cylinder length="0.11653" radius="0.16459"/>
+      </geometry>
+    </collision>
+  </link>
+  <joint name="rear_left_wheel" type="fixed">
+    <parent link="base_link"/>
+    <child link="rear_left_wheel_link"/>
+    <origin rpy="0 0 0" xyz="-0.249 0.29153 -0.0702"/>
+    <axis rpy="0 0 0" xyz="0 -1 0"/>
+  </joint>
+  <link name="rear_right_wheel_link">
+    <inertial>
+      <mass value="3"/>
+      <origin xyz="0 0 0"/>
+      <inertia ixx="0.7171" ixy="0" ixz="0" iyy="0.1361" iyz="0" izz="0.7171"/>
+    </inertial>
+    <visual>
+      <origin rpy="0 0 0" xyz="0 0 0"/>
+      <geometry>
+        <mesh filename="package://scout_description/meshes/scout_v2/wheel_type2.dae"/>
+      </geometry>
+    </visual>
+    <collision>
+      <origin rpy="1.570795 0 0" xyz="0 0 0"/>
+      <geometry>
+        <cylinder length="0.11653" radius="0.16459"/>
+      </geometry>
+    </collision>
+  </link>
+  <joint name="rear_right_wheel" type="fixed">
+    <parent link="base_link"/>
+    <child link="rear_right_wheel_link"/>
+    <origin rpy="3.14 0 0" xyz="-0.249 -0.29153 -0.0702"/>
+    <axis rpy="0 0 0" xyz="0 -1 0"/>
   </joint>
 </robot>
